Commit message: desenvolvimento do pacote moveit

File: src/spot_description/urdf/simple_robot.urdf (robot description, URDF)
Before this commit: robot simple_robot, 1 links, 0 joints
Links:
- removed link base_link
- added link base, mass 1.0; collision box size=0.1 0.1 0.1; visual mesh filename=/home/developer/SPWAR_ws/src/spot_description/meshes/base_l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

File: src/spot_description/urdf/spot_with_arm.urdf (robot description, URDF)
Before this commit: robot spot, 20 links, 19 joints
Links:
- link arm0.link_el0: geometry collision mesh filename=package://spot_description/meshes/arm0.link_el0.stl; visual mesh filename=package://spot_description/meshes/arm0.link_el0.stl
- link arm0.link_el1: geometry collision mesh filename=package://spot_description/meshes/arm0.link_el1.stl; visual mesh filename=package://spot_description/meshes/arm0.link_el1.stl
- link arm0.link_fngr: geometry collision mesh filename=package://spot_description/meshes/arm0.link_fngr.stl; visual mesh filename=package://spot_description/meshes/arm0.link_fngr.stl
- link arm0.link_sh0: geometry collision mesh filename=package://spot_description/meshes/arm0.link_sh0.stl; visual mesh filename=package://spot_description/meshes/arm0.link_sh0.stl
- link arm0.link_sh1: geometry collision mesh filename=package://spot_description/meshes/arm0.link_hr0.stl; collision mesh filename=package://spot_description/meshes/arm0.link_sh1.stl
- link arm0.link_wr0: geometry collision mesh filename=package://spot_description/meshes/arm0.link_wr0.stl; visual mesh filename=package://spot_description/meshes/arm0.link_wr0.stl
- link arm0.link_wr1: geometry collision mesh filename=package://spot_description/meshes/arm0.link_wr1.stl; visual mesh filename=package://spot_description/meshes/arm0.link_wr1.stl
