Commit message: codigo para verificação de pose e execução

File: src/spot_description/urdf/spot_with_arm.urdf (robot description, URDF)
Before this commit: robot spot, 20 links, 19 joints
Links:
- link base: mass 16.70765207 -> None
- link fl.hip: geometry collision mesh filename=package://spot_description/meshes/fl_hip_0_geom_visual_mesh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; visual mesh filename=package://spot_description/meshes/fl_hip_0_geom_visual_mesh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
- link fr.hip: geometry collision mesh filename=package://spot_description/meshes/fr_hip_0_geom_visual_mesh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; visual mesh filename=package://spot_description/meshes/fr_hip_0_geom_visual_mesh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
- link hl.hip: geometry collision mesh filename=package://spot_description/meshes/hl_hip_0_geom_visual_mesh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; visual mesh filename=package://spot_description/meshes/hl_hip_0_geom_visual_mesh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
- link hr.hip: geometry collision mesh filename=package://spot_description/meshes/hr_hip_0_geom_visual_mesh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; visual mesh filename=package://spot_description/meshes/hr_hip_0_geom_visual_mesh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

File: src/spot_moveit_config/config/spot.ros2_control.xacro (robot description, xacro)
@@ -2,5 +2,5 @@
 <robot xmlns:xacro="http://www.ros.org/wiki/xacro">
     <xacro:macro name="spot_ros2_control" params="name initial_positions_file">
-        <xacro:property name="initial_positions" value="${load_yaml(initial_positions_file)['initial_positions']}"/>
+        <xacro:property name="initial_positions" value="${xacro.load_yaml(initial_positions_file)['initial_positions']}"/>
         <ros2_control name="${name}" type="system">
             <hardware>
